Commit message: Add tongue and fix symmetric gripper

File: iai_wsg_50_description/urdf/wsg_50.urdf.xacro (robot description, xacro)
@@ -45,5 +45,4 @@
   <!-- GRIPPER LEFT -->
   <joint name="${name}_base_gripper_left_joint" type="prismatic">
-     <mimic joint ="${name}_joint" multiplier="-0.5"/>
      <limit lower="-0.055" upper="-0.0027" effort="1.0" velocity="0.42"/>
      <origin xyz="0 0 0" rpy="0 0 0" />      <!--origin xyz="-0.0067 0 0.049" rpy="0 0 0" /-->
@@ -130,8 +129,9 @@
   </gazebo>
   <!-- GRIPPER RIGHT -->
-  <joint name="${name}_joint" type="prismatic">
-     <limit lower="0.0065" upper="0.109" effort="1.0" velocity="0.42"/>
+  <joint name="${name}_base_gripper_right_joint" type="prismatic">
+    <mimic joint ="${name}_base_gripper_left_joint" multiplier="-1"/>
+     <limit lower="0.0027" upper="0.055" effort="1.0" velocity="0.42"/>
      <origin xyz="0 0 0" rpy="0 0 3.14159" />
-     <parent link="${name}_gripper_left_link"/>
+     <parent link="${name}_base_link"/>
      <child link="${name}_gripper_right_link" />
      <axis xyz="-1 0 0"/>
